File: fixtures/esp32_robot_carrier/esp32_robot_carrier_v3.kicad_pcb (KiCad board)
At the start: 2 copper layers, 128 x 189 mm, 157 parts, among them J3V3 3V3_AUX, J3V3_1 3V3_RAIL_1, J3V3_2 3V3_RAIL_2, J3V3_3 3V3_RAIL_3, J3V3_4 3V3_RAIL_4, Q5 STP100N10F7_100V, Q6 STP100N10F7_100V, U10 TLV9002IDR_DUAL_THROTTLE_RRIO, U4 LTC4367IMS8#PBF, U6 AQY212SX_60V_0.5A_PHOTOMOS, U7 AQY212SX_60V_0.5A_PHOTOMOS, U8 AQY212SX_60V_0.5A_PHOTOMOS, U9 AQY212SX_60V_0.5A_PHOTOMOS

Commit message: build: refresh hand-solder carrier fabrication
Parts:
- removed the U_RGB at (68.0, 102.5)
- removed the U_TRIG_F at (104.0, 40.0)
- removed the U_TRIG_L at (104.0, 10.0)
- removed the U_TRIG_R at (104.0, 46.0)
- added C28: 100nF_25V_AHCT125_BYPASS, C_1206_HAND_SOLDER, F.Cu at (145.0, 15.5)
- added U11: SN74AHCT125N_QUAD_3V3_TO_5V_BUFFER, DIP-14_W7.62mm_SN74AHCT125N_HAND_SOLDER, F.Cu at (139.0, 25.5)
- added U_RGB: DNP_TEST_ANCHOR_ONLY, DNP_BUFFER_TEST_ANCHOR, F.Cu at (68.0, 102.5)
- added U_TRIG_F: DNP_TEST_ANCHOR_ONLY, DNP_BUFFER_TEST_ANCHOR, F.Cu at (104.0, 40.0)
- added U_TRIG_L: DNP_TEST_ANCHOR_ONLY, DNP_BUFFER_TEST_ANCHOR, F.Cu at (104.0, 10.0)
- added U_TRIG_R: DNP_TEST_ANCHOR_ONLY, DNP_BUFFER_TEST_ANCHOR, F.Cu at (104.0, 46.0)
- C1, C2, C20, C27, C3: footprint C_0805_2012Metric -> C_1206_HAND_SOLDER
- C11, C18: footprint SMD2_1.15x2.7 -> C_1210_HAND_SOLDER
- C21, C22, C23: footprint R_0805_2012Metric -> C_1206_HAND_SOLDER
- C25: footprint C_1210_3225Metric -> C_1210_HAND_SOLDER
- R1, R10, R11, R12, R13, R14, R15, R16, R17, R18, R19, R2, R20, R21, R22, R23, R24, R25, R26, R27, R28, R29, R3, R30, R4, R40, R41, R42, R43, R44, R45, R46, R47, R48, R49, R5, R50, R51, R52, R53, R6, R7, R8, R9: footprint R_0805_2012Metric -> R_1206_HAND_SOLDER
- U10: footprint SOIC-8_3.9x4.9mm_P1.27mm_TLV9002 -> SOIC-8_TLV9002_HAND_SOLDER_LONG_PAD
- U4: footprint LTC4367_MSOP8 -> MSOP-8_LTC4367_HAND_SOLDER_LONG_PAD
- U6, U7, U8, U9: value AQY212SX_60V_0.5A_PHOTOMOS -> AQY212GH_60V_1.1A_PHOTOMOS; footprint Panasonic_AQY212S_SOP4 -> Panasonic_AQY212GH_DIP4_HAND_SOLDER
- moved U6 0.40 mm to (19.0, 38.0)
- moved U7 0.40 mm to (19.0, 44.0)
- moved U8 0.40 mm to (19.0, 62.0)
- moved U9 0.40 mm to (19.0, 68.0)
Routing:
- net RGB_DATA_5V: track 20.4 -> 153.1 mm, vias 0 -> 8
- net RIGHT_TRIG: track 27.6 -> 123.7 mm, vias 1 -> 5
- net RIGHT_TRIG_5V: track 7.02 -> 90.1 mm, vias 0 -> 2
- net FRONT_TRIG: track 28.4 -> 102.0 mm, vias 1 -> 5
- net FRONT_TRIG_5V: track 7.02 -> 75.7 mm, vias 0 -> 3
- net LEFT_TRIG: track 44.3 -> 110.1 mm
- net +5V: track 441.8 -> 494.5 mm, vias 6 -> 8
- net LEFT_TRIG_5V: track 7.02 -> 50.8 mm
- net AUX_GPIO2: track 208.8 -> 228.8 mm
- net GND: track 144.5 -> 147.6 mm
- net L_THROTTLE_FILTERED: track 94.1 -> 95.7 mm
- net R_REVERSE_CONTACT_B: track 12.3 -> 13.8 mm
- net R_REVERSE_CONTACT_A_SW: track 3.48 -> 5.04 mm
- net R_BRAKE_CONTACT_B: track 13.2 -> 14.8 mm
- net R_BRAKE_CONTACT_A_SW: track 3.48 -> 5.04 mm
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Other:
- board size 128 x 189 mm -> 155 x 189 mm
- board text added: "HAND-SOLDER BUILD | 1206 + DIP"
- board text removed: "L BRK EN"
- board text removed: "L GND"
- board text removed: "R BRK EN"
- board text removed: "R GND"
- board text removed: "R REV EN"
